File: kicad_files/austin.kicad_sch (KiCad schematic)
At the start: 559 parts, among them J1 EXTRA PINS, J2 ARM SWD, J3 TYPE-C-31-M-12, Q1 DTC123JKAT146, Q2 AO3401A, Q3 DTC123JKAT146, SW1 K2-1187SQ-A4SW-06, SW10 MXSwitch, SW100 MXSwitch, SW101 MXSwitch, SW102 MXSwitch, SW103 MXSwitch, SW104 MXSwitch, SW105 MXSwitch, SW106 MXSwitch, SW107 MXSwitch, SW108 MXSwitch, SW109 MXSwitch, SW11 MXSwitch, SW110 MXSwitch, SW111 MXSwitch, SW112 MXSwitch, SW113 MXSwitch, SW114 MXSwitch, SW115 MXSwitch, SW116 MXSwitch, SW12 MXSwitch, SW13 MXSwitch, SW14 MXSwitch, SW15 MXSwitch, SW16 MXSwitch, SW17 MXSwitch, SW18 MXSwitch, SW19 MXSwitch, SW2 PCM12SMTR, SW20 MXSwitch, SW21 MXSwitch, SW22 MXSwitch, SW23 MXSwitch, SW24 MXSwitch, SW25 MXSwitch, SW26 MXSwitch, SW27 MXSwitch, SW28 MXSwitch, SW29 MXSwitch, SW3 MXSwitch, SW30 MXSwitch, SW31 MXSwitch, SW32 MXSwitch, SW33 MXSwitch, SW34 MXSwitch, SW35 MXSwitch, SW36 MXSwitch, SW37 MXSwitch, SW38 MXSwitch, SW39 MXSwitch, SW4 MXSwitch, SW40 MXSwitch, SW41 MXSwitch, SW42 MXSwitch, SW43 MXSwitch, SW44 MXSwitch, SW45 MXSwitch, SW46 MXSwitch, SW47 MXSwitch, SW48 MXSwitch, SW49 MXSwitch, SW5 MXSwitch, SW50 MXSwitch, SW51 MXSwitch, SW52 MXSwitch, SW53 MXSwitch, SW54 MXSwitch, SW55 MXSwitch, SW56 MXSwitch, SW57 MXSwitch, SW58 MXSwitch, SW59 MXSwitch, SW6 MXSwitch, SW60 MXSwitch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

Commit message: Added MCU, reset, LDO circuits
Parts:
- removed C1: 1u, Capacitor_SMD:C_0402_1005Metric, symbol Device:C_Small
- removed C2: 100n, Capacitor_SMD:C_0402_1005Metric, symbol Device:C_Small
- removed C3, C4: 1u, acheronComponents:CP_EIA-3216-10_Kemet-I_Pad1.58x1.35mm_HandSolder, symbol Device:CP_Small
- removed C9: 10n, Capacitor_SMD:C_0402_1005Metric, symbol Device:C_Small
- removed D1: RB060M-60TR, acheronComponents:D_SOD-123, symbol Device:D
- removed D2: SMF6.0A, acheronComponents:D_SOD-123, symbol Device:D_Schottky
- removed D3: 1N4148W, acheronComponents:D_SOD-123, symbol Device:D
- removed F1: RF1338-000, acheronComponents:Fuse_1812_4532, symbol Device:Polyfuse_Small
- removed J1: EXTRA PINS, acheronConnectors:PinHeader_1x4_P2.54mm_Vertical, symbol Connector_Generic:Conn_01x04
- removed J2: ARM SWD, acheronConnectors:Conn_ARM_JTAG_SWD_8, symbol Connector_Generic:Conn_02x04_Odd_Even
- removed LED63: LED, acheronComponents:LED_THT_2.54mm, symbol austin-rescue:LED-acheronSymbols-austin-rescue-austin-rescue
- removed Q1: DTC123JKAT146, Package_TO_SOT_SMD:SOT-23, symbol Transistor_BJT:DTC123J
- removed R109: 470R, Resistor_SMD:R_0805_2012Metric, symbol Device:R_Small
- removed R3: 100k, Resistor_SMD:R_0805_2012Metric, symbol Device:R
- removed SW1: K2-1187SQ-A4SW-06, acheronHardware:K2-1187SQ-A4SW-06, symbol Switch:SW_Push
- removed U1: MCP1700T-3302E/TT, Package_TO_SOT_SMD:SOT-23, symbol Regulator_Linear:MCP1700-3302E_SOT23
- removed U2: STM32F072CBT6, acheronComponents:LQFP48_UFQFPN48_7x7mm_P0.5mm, symbol acheronSymbols:STM32F072-UFQFPN48
- added C1, C2: 1u, Capacitor_SMD:C_0805_2012Metric, symbol Device:C
- added C14, C15: 100n, Capacitor_SMD:C_0402_1005Metric, symbol Device:C_Small
- added C16: 4.7u, Capacitor_SMD:C_0402_1005Metric, symbol Device:C_Small
- added C3: 10n, Capacitor_SMD:C_0402_1005Metric, symbol Device:C_Small
- added C4: 10u, Capacitor_SMD:C_0402_1005Metric, symbol Device:C_Small
- added C9: 10u, acheron_Components:CP_EIA-3216-10_Kemet-I_Pad1.58x1.35mm_HandSolder, symbol Device:CP1
- added D1: B5819W-SL, acheron_Components:D_SOD-123, symbol Device:D_Schottky
- added D2: 1N4148W, acheron_Components:D_SOD-123, symbol Device:D
- added R1: 100k, Resistor_SMD:R_0805_2012Metric, symbol Device:R
- added R11, R12: 4.7k, Resistor_SMD:R_0402_1005Metric, symbol Device:R_Small
- added R13: 1.5k, Resistor_SMD:R_0402_1005Metric, symbol Device:R_Small
- added R3: 330k, Resistor_SMD:R_0402_1005Metric, symbol Device:R_Small
- added R4: 1M, Resistor_SMD:R_0402_1005Metric, symbol Device:R_Small
- added R5: 10k, Resistor_SMD:R_0402_1005Metric, symbol Device:R_Small
- added R6, R7: 100R, Resistor_SMD:R_0402_1005Metric, symbol Device:R_Small
- added SW1: K2-1187SQ-A4SW-06, acheron_Hardware:K2-1187SQ-A4SW-06, symbol Switch:SW_SPST
- added U1: SPX3819M5-L-3-3, acheron_Components:SOT-23-5, symbol acheron_Symbols:SGM2036
- added U2: 2N7002DW, acheron_Components:SOT-363_SC-70-6, symbol acheron_Symbols:2N7002DW
- added U3: STM32F401RCT6, acheron_Components:LQFP-64_10x10mm_P0.5mm, symbol acheron_Symbols:STM32F401-LQFP64
- added X1, X2: ARM JTAG, acheron_Connectors:PinHeader_2x5_P2.54mm_Vertical_Staggered, symbol Connector_Generic:Conn_02x05_Odd_Even
- added Y1: TAXM8M4RFDCET2T, acheron_Components:Crystal_SMD_3225-4Pin_3.2x2.5mm, symbol Device:Crystal_GND24
- C10: value 100n -> 15p; Manufacturer (none) -> Guangdong Fenghua Advanced Tech; Manufacturer Part Number (none) -> 0402CG150J500NT; Specification (none) -> 50V 15pF C0G ±5% 0402 MLCC; Vendor Part Number (none) -> LCSC C1548
- C11: value 1u -> 15p; Manufacturer (none) -> Guangdong Fenghua Advanced Tech; Manufacturer Part Number (none) -> 0402CG150J500NT; Specification (none) -> 50V 15pF C0G ±5% 0402 MLCC; Vendor Part Number (none) -> LCSC C1548
- C12: value 10n -> 4.7u; footprint Capacitor_SMD:C_0805_2012Metric -> Capacitor_SMD:C_0402_1005Metric; Manufacturer (none) -> Samsung; Manufacturer Part Number (none) -> CL05A475MP5NRNC; Specification (none) -> 10V 4.7uF X5R ±20% 0402 MLCC; Vendor Part Number (none) -> LCSC C23733
- C13: value 10u -> 10n; footprint Capacitor_SMD:C_0805_2012Metric -> Capacitor_SMD:C_0402_1005Metric; Manufacturer (none) -> Samsung; Manufacturer Part Number (none) -> CL05B103KB5NNNC; Specification (none) -> 50V 10nF X7R ±10% 0402 MLCC; Vendor Part Number (none) -> LCSC C15195
- C5, C6: Manufacturer (none) -> Samsung; Manufacturer Part Number (none) -> CL05B104KB54PNC; Specification (none) -> 50V 100nF X7R ±10% 0402 MLCC; Vendor Part Number (none) -> LCSC C307331
- C7: value 1u -> 100n; Manufacturer (none) -> Samsung; Manufacturer Part Number (none) -> CL05B104KB54PNC; Specification (none) -> 50V 100nF X7R ±10% 0402 MLCC; Vendor Part Number (none) -> LCSC C307331
- C8: value 4.7u -> 100n; Manufacturer (none) -> Samsung; Manufacturer Part Number (none) -> CL05B104KB54PNC; Specification (none) -> 50V 100nF X7R ±10% 0402 MLCC; Vendor Part Number (none) -> LCSC C307331
- D10: renamed from D11; footprint acheronComponents:LED_WS2812B_5.0x5.0mm_P3.2mm -> acheron_Components:LED_WS2812B_5.0x5.0mm_P3.2mm
- D100: renamed from D101; footprint acheronComponents:D_SOD-123 -> acheron_Components:D_SOD-123
- D101: renamed from D102; footprint acheronComponents:D_SOD-123 -> acheron_Components:D_SOD-123
- D102: renamed from D103; footprint acheronComponents:D_SOD-123 -> acheron_Components:D_SOD-123
- D103: renamed from D104; footprint acheronComponents:D_SOD-123 -> acheron_Components:D_SOD-123
- D104: renamed from D105; footprint acheronComponents:D_SOD-123 -> acheron_Components:D_SOD-123
- D105: renamed from D106; footprint acheronComponents:D_SOD-123 -> acheron_Components:D_SOD-123
- D106: renamed from D107; footprint acheronComponents:D_SOD-123 -> acheron_Components:D_SOD-123
- D107: renamed from D108; footprint acheronComponents:D_SOD-123 -> acheron_Components:D_SOD-123
- D108: renamed from D109; footprint acheronComponents:D_SOD-123 -> acheron_Components:D_SOD-123
- D109: renamed from D110; footprint acheronComponents:D_SOD-123 -> acheron_Components:D_SOD-123
- D11: renamed from D12; footprint acheronComponents:LED_WS2812B_5.0x5.0mm_P3.2mm -> acheron_Components:LED_WS2812B_5.0x5.0mm_P3.2mm
- D110: renamed from D111; footprint acheronComponents:D_SOD-123 -> acheron_Components:D_SOD-123
- D111: renamed from D112; footprint acheronComponents:D_SOD-123 -> acheron_Components:D_SOD-123
- D112: renamed from D113; footprint acheronComponents:D_SOD-123 -> acheron_Components:D_SOD-123
- D113: renamed from D114; footprint acheronComponents:D_SOD-123 -> acheron_Components:D_SOD-123
- D114: renamed from D115; footprint acheronComponents:D_SOD-123 -> acheron_Components:D_SOD-123
- D115: renamed from D116; footprint acheronComponents:D_SOD-123 -> acheron_Components:D_SOD-123
- D116: renamed from D117; footprint acheronComponents:D_SOD-123 -> acheron_Components:D_SOD-123
- D117: renamed from D118; footprint acheronComponents:D_SOD-123 -> acheron_Components:D_SOD-123
- D118: renamed from D119; footprint acheronComponents:D_SOD-123 -> acheron_Components:D_SOD-123
- D119: renamed from D120; footprint acheronComponents:D_SOD-123 -> acheron_Components:D_SOD-123
- D12: renamed from D13; footprint acheronComponents:LED_WS2812B_5.0x5.0mm_P3.2mm -> acheron_Components:LED_WS2812B_5.0x5.0mm_P3.2mm
- D120: renamed from D121; footprint acheronComponents:D_SOD-123 -> acheron_Components:D_SOD-123
- D121: renamed from D122; footprint acheronComponents:D_SOD-123 -> acheron_Components:D_SOD-123
- D122: renamed from D123; footprint acheronComponents:D_SOD-123 -> acheron_Components:D_SOD-123
- D123: renamed from D124; footprint acheronComponents:D_SOD-123 -> acheron_Components:D_SOD-123
- D124: renamed from D125; footprint acheronComponents:D_SOD-123 -> acheron_Components:D_SOD-123
- D125: renamed from D126; footprint acheronComponents:D_SOD-123 -> acheron_Components:D_SOD-123
- D126: renamed from D127; footprint acheronComponents:D_SOD-123 -> acheron_Components:D_SOD-123
- D127: renamed from D128; footprint acheronComponents:D_SOD-123 -> acheron_Components:D_SOD-123
- D13: renamed from D14; footprint acheronComponents:LED_WS2812B_5.0x5.0mm_P3.2mm -> acheron_Components:LED_WS2812B_5.0x5.0mm_P3.2mm
- D14: renamed from D15; footprint acheronComponents:LED_WS2812B_5.0x5.0mm_P3.2mm -> acheron_Components:LED_WS2812B_5.0x5.0mm_P3.2mm
- D15: renamed from D16; footprint acheronComponents:LED_WS2812B_5.0x5.0mm_P3.2mm -> acheron_Components:LED_WS2812B_5.0x5.0mm_P3.2mm
- D16: renamed from D17; footprint acheronComponents:LED_WS2812B_5.0x5.0mm_P3.2mm -> acheron_Components:LED_WS2812B_5.0x5.0mm_P3.2mm
- D17: renamed from D18; footprint acheronComponents:LED_WS2812B_5.0x5.0mm_P3.2mm -> acheron_Components:LED_WS2812B_5.0x5.0mm_P3.2mm
- D18: renamed from D19; footprint acheronComponents:LED_WS2812B_5.0x5.0mm_P3.2mm -> acheron_Components:LED_WS2812B_5.0x5.0mm_P3.2mm
- D19: renamed from D20; footprint acheronComponents:LED_WS2812B_5.0x5.0mm_P3.2mm -> acheron_Components:LED_WS2812B_5.0x5.0mm_P3.2mm
- D20: renamed from D21; footprint acheronComponents:LED_WS2812B_5.0x5.0mm_P3.2mm -> acheron_Components:LED_WS2812B_5.0x5.0mm_P3.2mm
- D21: renamed from D22; footprint acheronComponents:LED_WS2812B_5.0x5.0mm_P3.2mm -> acheron_Components:LED_WS2812B_5.0x5.0mm_P3.2mm
- D22: renamed from D23; footprint acheronComponents:LED_WS2812B_5.0x5.0mm_P3.2mm -> acheron_Components:LED_WS2812B_5.0x5.0mm_P3.2mm
- D23: renamed from D24; footprint acheronComponents:D_SOD-123 -> acheron_Components:D_SOD-123
- D24: renamed from D25; footprint acheronComponents:D_SOD-123 -> acheron_Components:D_SOD-123
- D25: renamed from D26; footprint acheronComponents:D_SOD-123 -> acheron_Components:D_SOD-123
- D26: renamed from D27; footprint acheronComponents:D_SOD-123 -> acheron_Components:D_SOD-123
- D27: renamed from D28; footprint acheronComponents:D_SOD-123 -> acheron_Components:D_SOD-123
- D28: renamed from D29; footprint acheronComponents:D_SOD-123 -> acheron_Components:D_SOD-123
- D29: renamed from D30; footprint acheronComponents:D_SOD-123 -> acheron_Components:D_SOD-123
- D3: renamed from D4; footprint acheronComponents:LED_WS2812B_5.0x5.0mm_P3.2mm -> acheron_Components:LED_WS2812B_5.0x5.0mm_P3.2mm
- D30: renamed from D31; footprint acheronComponents:D_SOD-123 -> acheron_Components:D_SOD-123
- renumbered C14 to C17, C15 to C18, C16 to C19, C17 to C20, C18 to C21, C19 to C22, C20 to C23, C21 to C24, C22 to C25, C23 to C26, C24 to C27, C25 to C28, C26 to C29, C27 to C30, C28 to C31, C29 to C32, C30 to C33, C31 to C34, C32 to C35, C33 to C36, C34 to C37, C35 to C38, Q2 to Q1, Q3 to Q2, R11 to R19, R12 to R20, R13 to R21, R14 to R22, R15 to R23, R16 to R24, R17 to R25, R18 to R26, R19 to R27, R20 to R28, R21 to R29, R22 to R30, R23 to R31, R24 to R32, R25 to R33, R26 to R34, R27 to R35, R28 to R36, R29 to R37, R30 to R38, R31 to R39, R33 to R40, R34 to R41, SW2 to SW61
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Connections:
- net 3V3: now also C12.2, C13.2, C7.1, C8.1, R2.1, C14.2, C15.1, C2.1, C9.1, D1.2 (A), R11.2, R12.2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; no longer C10.2, C11.2, C5.1, C7.2, C8.2
- net 5V: now also C1.1, D1.1 (K), R1.1, U1.1 (IN), U1.3 (EN); no longer R2.1
- net BOOT0: now also C4.1, R3.1, R4.1, R5.2, U3.60 (BOOT0), X1.5 (Pin_5), X2.5 (Pin_5); no longer C13.2, R10.1, R9.2
- net D+: now also R13.1, U3.45 (OTG_FS_DP/USART6_RX/PA12)
- net D-: now also U3.44 (OTG_FS_DM/TIM1_CH4/USART6_TX/PA11)
- net GND: now also C10.2, C11.2, C12.1, C7.2, C8.2, R9.1, C1.2, C14.1, C15.2, C16.1, C2.2, C3.1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; no longer C10.1, C11.1, C12.2, C7.1, C8.1
- net LED_PWM: now also U3.56 (NJTRST/SPI1_MISO/SPI3_MISO/I2C3_SDA/TIM3_CH1/PB4)
- net NRST: now also C5.1, R7.2, U3.7 (NRST), X1.9 (Pin_9), X2.9 (Pin_9); no longer C12.1, R8.2
- net RGB_3V3: now also U3.36 (SPI2_MOSI/PB15)
- net SWCLK: now also U3.49 (JTCK-SWCLK/PA14), X1.2 (Pin_2), X2.2 (Pin_2)
- net SWDIO: now also U3.46 (JTMS-SWDIO/PA13), X1.1 (Pin_1), X2.1 (Pin_1)
- net at R8.1: now also R9.2, U2.2 (G)
- new net: R6.2, R7.1, U2.6 (D)
- new net: D2.2 (A), R8.2, SW1.2 (B)
- new net: C16.2, U3.30 (VCAP1)
- new net: D2.1 (K), R3.2
- new net: R6.1, U2.5 (G)
- new net: C3.2, U1.4 (BP/FB)
- new net: R5.1, U2.3 (D)
- new net C0: U3.41 (USART1_CK/TIM1_CH1/PA8)
- new net C1: U3.40 (TIM3_CH4/I2S_CKIN/PC9)
- new net C10: U3.52 (SPI3_MISO/PC11)
- new net C11: U3.53 (SPI3_MOSI/PC12)
- new net C12: U3.54 (PD2)
- new net C13: U3.55 (JTDO-SWO/SPI1_SCK/SPI3_SCK/I2C2_SDA/TIM2_CH2/PB3)
- new net C14: U3.57 (SPI1_MOSI/SPI3_MOSI/TIM3_CH2/PB5)
- new net C2: U3.39 (USART6_CK/TIM3_CH3/PC8)
- new net C3: U3.38 (USART6_RX/TIM3_CH2/PC7)
- new net C4: U3.37 (I2S2_MCK/TIM3_CH1/USART6_TX/PC6)
- new net C5: U3.8 (PC0)
- new net C6: U3.62 (I2C1_SDA/TIM4_CH4/TIM11_CH1/PB9)
- new net C7: U3.11 (PC3/SPI2_MOSI)
- new net C8: U3.50 (JTDI/TIM2_CH1/PA14)
- new net C9: U3.51 (SPI3_SCK/I2S3_CK/PC10)
- new net CAPS_INDICATOR: U3.43 (USART1_RX/TIM1_CH3/PA10)
- new net E-PA9: U3.42 (USART1_TX/TIM1_CH2/PA9)
- new net E-PB0: U3.26 (PB0/TIM3_CH3)
- new net E-PB1: U3.27 (PB1/TIM3_CH4)
- new net E-PB10: U3.29 (PB10/TIM2_CH3/SPI2_SCK/I2C2_SCL/I2S2_CK)
- new net E-PB12: U3.33 (PB12)
- new net E-PB13: U3.34 (SPI2_SCK/I2S2_CK/PB13)
- new net E-PB14: U3.35 (SPI2_MISO/PB14)
- new net E-PC13: U3.2 (PC13)
- new net E-PC14: U3.3 (PC14/OSC32_IN)
- new net E-PC15: U3.4 (PC15/OSC32_OUT)
- new net E-PC4: U3.24 (PC4)
- new net E-PC5: U3.25 (PC5)
- new net PB2/BOOT1: R10.1, U3.28 (PB2), X1.6 (Pin_6), X2.6 (Pin_6)
- new net R0: U3.23 (PA7/SPI1_MOSI/TIM3_CH2)
- new net R1: U3.9 (PC1)
- new net R10: U3.17 (PA3/TIM2_CH4/USART2_RX)
- new net R2: U3.22 (PA6/TIM3_CH1/SPI1_MISO)
- new net R3: U3.21 (PA5/TIM2_CH1/SPI1_SCK)
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Other:
- note added: "(*) "Spooky pins": on STM32F4x1, pins A9 and B2 cannot be used for switch matrix: - A9 is meant to be used as a VBUS sensing. It has a undocumented internal pulldown resistor; - B2 is used as BOOT1 during bootup, so it needs an external pulldown for successful bootup"
- note added: "(**) PA9 jumper: a solderable jumper used to tie PA9 to VBUS. It is disconnected by default, hence PA9 is left floating"
- note added: "3V3"
- note added: "HARD RESET"
- note added: "SPOOKY PIN"
- note removed: "Hard reset circuit"
- note removed: "Power supply and protection circuit"

Commit message: Routing
Parts:
- removed Q2: DTC123JKAT146, Package_TO_SOT_SMD:SOT-23, symbol acheronSymbols:DTC123J
- removed R40: 1k, Resistor_SMD:R_0805_2012Metric, symbol Device:R
- removed R41: 100R, Resistor_SMD:R_0805_2012Metric, symbol Device:R
- removed SW61: PCM12SMTR, Button_Switch_SMD:SW_SPDT_PCM12, symbol Switch:SW_SPDT
- added Q2, Q3: 2N7002, Package_TO_SOT_SMD:SOT-23, symbol Transistor_FET:2N7002
- added R100, R40, R43: 10k, Resistor_SMD:R_0402_1005Metric, symbol Device:R_Small
- added R41, R42, R83: 100, Resistor_SMD:R_0402_1005Metric, symbol Device:R_Small
- C17, C18, C19, C20, C21, C22, C23, C24, C25, C26, C27, C28, C29, C30, C31, C32, C33, C34, C35, C36, C37, C38: footprint Capacitor_SMD:C_0805_2012Metric -> Capacitor_SMD:C_0402_1005Metric; Package C0805 -> C0402
- Q1: LCSC Part Number C15127 -> (none); Manufacturer Alpha and Omega Semicon -> AO3401A; Manufacturer Part Number AO3401A -> Alpha & Omega Semicon; Specification (none) -> P-channel power MOSFET transistor; Vendor Part Number (none) -> LCSC C15127
- R19, R20, R21, R22, R23, R24, R25, R26, R27, R28, R29, R30, R31, R32, R33, R34, R35, R36, R37, R38: value 4.7R -> 5.1R; footprint Resistor_SMD:R_0805_2012Metric -> Resistor_SMD:R_0402_1005Metric; Package R0805 -> R0402
- R39: footprint Resistor_SMD:R_0805_2012Metric -> Resistor_SMD:R_0402_1005Metric; Package R0805 -> R0402
- renumbered LED10 to LED1, LED7 to LED10, LED8 to LED11, LED9 to LED12, LED11 to LED2, LED42 to LED20, LED43 to LED21, LED20 to LED22, LED21 to LED23, LED22 to LED24, LED23 to LED25, LED24 to LED26, LED25 to LED27, LED26 to LED28, LED27 to LED29, LED12 to LED3, LED28 to LED30, LED29 to LED31, LED30 to LED32, LED31 to LED33, LED32 to LED34, LED33 to LED35, LED34 to LED36, LED35 to LED37, LED36 to LED38, LED37 to LED39, LED1 to LED4, LED38 to LED40, LED39 to LED41, LED40 to LED42, LED61 to LED43, LED41 to LED44, LED44 to LED45, LED45 to LED46, LED46 to LED47, LED47 to LED48, LED48 to LED49, LED2 to LED5, LED49 to LED50, LED50 to LED51, LED51 to LED52, LED52 to LED53, LED53 to LED54, LED54 to LED55, LED55 to LED56, LED56 to LED57, LED57 to LED58, LED58 to LED59, LED3 to LED6, LED59 to LED60, LED60 to LED61, LED4 to LED7, LED5 to LED8, LED6 to LED9, R97 to R101, R96 to R102, R98 to R103, R100 to R104, R101 to R105, R102 to R106, R103 to R107, R104 to R108, R105 to R109, R106 to R110, R107 to R111, R108 to R112, R109 to R113, R110 to R114, R111 to R115, R112 to R116, R113 to R117, R114 to R118, R115 to R119, R116 to R120, R117 to R121, R118 to R122, R119 to R123, R120 to R124, R121 to R125, R122 to R126, R123 to R127, R124 to R128, R125 to R129, R126 to R130, R127 to R131, R128 to R132, R129 to R133, R130 to R134, R131 to R135, R132 to R136, R133 to R137, R134 to R138, R135 to R139, R136 to R140, R137 to R141, R138 to R142, R139 to R143, R140 to R144, R141 to R145, R142 to R146, R143 to R147, R144 to R148, R145 to R149, R146 to R150, R147 to R151, R42 to R44, R43 to R45, R44 to R46, R45 to R47, R46 to R48, R47 to R49, R48 to R50, R49 to R51, R53 to R52, R54 to R53, R55 to R54, R56 to R55, R57 to R56, R58 to R57, R59 to R58, R50 to R59, R51 to R60, R52 to R61, R60 to R62, R61 to R63, R62 to R64, R63 to R65, R64 to R66, R65 to R67, R66 to R68, R67 to R69, R68 to R70, R69 to R71, R70 to R72, R71 to R73, R72 to R74, R73 to R75, R74 to R76, R75 to R77, R76 to R78, R77 to R79, R99 to R80, R78 to R81, R79 to R82, R80 to R84, R81 to R85, R82 to R86, R83 to R87, R84 to R88, R85 to R89, R86 to R90, R87 to R91, R88 to R92, R89 to R93, R90 to R94, R91 to R95, R92 to R96, R93 to R97, R94 to R98, R95 to R99, SW101 to SW100, SW102 to SW101, SW103 to SW102, SW104 to SW103, SW105 to SW104, SW106 to SW105, SW107 to SW106, SW108 to SW107, SW109 to SW108, SW110 to SW109, SW111 to SW110, SW112 to SW111, SW113 to SW112, SW114 to SW113, SW115 to SW114, SW116 to SW115, SW62 to SW61, SW63 to SW62, SW64 to SW63, SW65 to SW64, SW66 to SW65, SW67 to SW66, SW68 to SW67, SW69 to SW68, SW70 to SW69, SW71 to SW70, SW72 to SW71, SW73 to SW72, SW74 to SW73, SW75 to SW74, SW76 to SW75, SW77 to SW76, SW78 to SW77, SW79 to SW78, SW80 to SW79, SW81 to SW80, SW82 to SW81, SW83 to SW82, SW84 to SW83, SW85 to SW84, SW86 to SW85, SW87 to SW86, SW88 to SW87, SW89 to SW88, SW90 to SW89, SW91 to SW90, SW92 to SW91, SW93 to SW92, SW94 to SW93, SW95 to SW94, SW96 to SW95, SW97 to SW96, SW98 to SW97, SW99 to SW98, SW100 to SW99
Connections:
- net Col1 is gone; now on net C0: SW100.1, SW110.1, SW2.2, SW21.2, SW42.1, SW62.2, SW80.1, SW81.1, SW83.1
- net Col10 is gone; now on net C9: SW11.2, SW30.1, SW51.1, SW71.1, SW92.1
- net Col11 is gone; now on net C10: SW103.1, SW12.1, SW31.1, SW52.1, SW72.1, SW93.1
- net Col12 is gone; now on net C11: SW104.1, SW13.1, SW32.1, SW53.1, SW73.1, SW94.1
- net Col13 is gone; now on net C12: SW105.1, SW14.1, SW33.1, SW54.1, SW61.1, SW74.1, SW82.1
- net Col14 is gone; now on net C13: SW106.1, SW15.1, SW34.1, SW41.1, SW55.1, SW75.1, SW95.1
- net Col15 is gone; now on net C14: SW114.1, SW16.1, SW35.1, SW40.1, SW56.1, SW76.1, SW96.1
- net Col3 is gone; now on net C2: SW112.1, SW23.1, SW4.1, SW44.1, SW64.1, SW85.1
- net Col4 is gone; now on net C3: SW24.1, SW45.1, SW5.1, SW65.1, SW86.1
- net Col5 is gone; now on net C4: SW25.1, SW46.1, SW6.1, SW66.1, SW87.1
- net Col7 is gone; now on net C6: SW27.1, SW48.1, SW68.1, SW8.1, SW89.1
- net Col8 is gone; now on net C7: SW28.1, SW49.1, SW69.1, SW9.1, SW90.1
- net E-PB1 is gone; now on net LED_PWM: U3.27 (PB1/TIM3_CH4)
- net E-PB12 is gone; now on net C7: U3.33 (PB12)
- net R10 is gone; now on net C2: U3.17 (PA3/TIM2_CH4/USART2_RX)
- net R7 is gone; now on net C5: U3.14 (PA0/TIM2_CH1/USART2_CTS)
- net R8 is gone; now on net C4: U3.15 (PA1/TIM2_CH2/USART2_RTS)
- net R9 is gone; now on net C3: U3.16 (PA2/TIM2_CH3/USART2_TX)
- net Row1 is gone; now on net R0: D23.1 (K), D24.1 (K), D25.1 (K), D26.1 (K), D27.1 (K), D28.1 (K), D29.1 (K), D30.1 (K), D31.1 (K), D32.1 (K), D33.1 (K), D34.1 (K), D35.1 (K), D36.1 (K), D37.1 (K), D38.1 (K), D39.1 (K), D40.1 (K), D41.1 (K)
- net Row2 is gone; now on net R1: D42.1 (K), D43.1 (K), D44.1 (K), D45.1 (K), D46.1 (K), D47.1 (K), D48.1 (K), D49.1 (K), D50.1 (K), D51.1 (K), D52.1 (K), D53.1 (K), D54.1 (K), D55.1 (K), D56.1 (K), D57.1 (K), D58.1 (K), D59.1 (K), D60.1 (K)
- net Row3 is gone; now on net R2: D61.1 (K), D62.1 (K), D63.1 (K), D64.1 (K), D65.1 (K), D66.1 (K), D67.1 (K), D68.1 (K), D69.1 (K), D70.1 (K), D71.1 (K), D72.1 (K), D73.1 (K), D74.1 (K), D75.1 (K), D76.1 (K), D77.1 (K), D78.1 (K), D79.1 (K)
- net Row4 is gone; now on net R3: D80.1 (K), D81.1 (K), D82.1 (K), D83.1 (K), D84.1 (K), D85.1 (K), D86.1 (K), D87.1 (K), D88.1 (K), D89.1 (K), D90.1 (K), D91.1 (K), D92.1 (K), D93.1 (K), D94.1 (K), D95.1 (K), D96.1 (K), D97.1 (K)
- net Row5 is gone; now on net R4: D100.1 (K), D101.1 (K), D102.1 (K), D103.1 (K), D104.1 (K), D105.1 (K), D106.1 (K), D107.1 (K), D108.1 (K), D109.1 (K), D110.1 (K), D111.1 (K), D112.1 (K), D113.1 (K), D114.1 (K), D115.1 (K), D98.1 (K), D99.1 (K)
- net Row6 is gone; now on net R5: D116.1 (K), D117.1 (K), D118.1 (K), D119.1 (K), D120.1 (K), D121.1 (K), D122.1 (K), D123.1 (K), D124.1 (K), D125.1 (K), D126.1 (K), D127.1 (K)
- net 5V: now also R40.2
- net C0: now also U3.21 (PA5/TIM2_CH1/SPI1_SCK); no longer U3.41 (USART1_CK/TIM1_CH1/PA8)
- net C1: now also SW101.1, SW111.2, SW22.1, SW3.1, SW43.1, SW63.1, SW84.2, U3.20 (PA4/USART2_CK); no longer U3.40 (TIM3_CH4/I2S_CKIN/PC9)
- net C10: no longer U3.52 (SPI3_MISO/PC11)
- net C11: no longer U3.53 (SPI3_MOSI/PC12)
- net C12: no longer U3.54 (PD2)
- net C13: no longer U3.55 (JTDO-SWO/SPI1_SCK/SPI3_SCK/I2C2_SDA/TIM2_CH2/PB3)
- net C14: no longer U3.57 (SPI1_MOSI/SPI3_MOSI/TIM3_CH2/PB5)
- net C2: no longer U3.39 (USART6_CK/TIM3_CH3/PC8)
- net C3: no longer U3.38 (USART6_RX/TIM3_CH2/PC7)
- net C4: no longer U3.37 (I2S2_MCK/TIM3_CH1/USART6_TX/PC6)
- net C5: now also SW102.1, SW113.2, SW26.1, SW47.1, SW67.1, SW7.1, SW88.1; no longer U3.8 (PC0)
- net C6: now also U3.37 (I2S2_MCK/TIM3_CH1/USART6_TX/PC6); no longer U3.62 (I2C1_SDA/TIM4_CH4/TIM11_CH1/PB9)
- net C7: no longer U3.11 (PC3/SPI2_MOSI)
- net C8: now also SW10.1, SW29.1, SW50.1, SW70.1, SW91.2, U3.41 (USART1_CK/TIM1_CH1/PA8); no longer U3.50 (JTDI/TIM2_CH1/PA14)
- net C9: now also U3.40 (TIM3_CH4/I2S_CKIN/PC9); no longer U3.51 (SPI3_SCK/I2S3_CK/PC10)
- net GND: now also R102.2, R59.2, R60.2, R61.2, Q2.2 (S), Q3.2 (S), R100.1, R43.1; no longer LED1.K, LED2.K, LED3.K, LED43.K
- net INDICATOR3: now also U3.38 (USART6_RX/TIM3_CH2/PC7), R83.1
- net LED_PWM: now also R42.1; no longer U3.56 (NJTRST/SPI1_MISO/SPI3_MISO/I2C3_SDA/TIM3_CH1/PB4)
- net LED_SIGNAL: now also LED1.A, LED2.A, LED3.A, LED43.A, R63.2, R64.2, R65.2, R66.2, R67.2, R68.2, R69.2, R70.2, R71.2, R72.2, R73.2, R74.2; no longer R102.1, R59.1, R60.1, R61.1, R63.1, R64.1, R65.1, R66.1, R67.1, R68.1, R69.1, R70.1, R71.1, R72.1, R73.1, R74.1
- net R0: no longer U3.23 (PA7/SPI1_MOSI/TIM3_CH2)
- net R1: no longer U3.9 (PC1)
- net R2: no longer U3.22 (PA6/TIM3_CH1/SPI1_MISO)
- net R3: no longer U3.21 (PA5/TIM2_CH1/SPI1_SCK)
- net R4: no longer U3.20 (PA4/USART2_CK)
- net R5: no longer U3.61 (I2C1_SCL/TIM4_CH3/TIM10_CH1/PB8)
- net at D28.2 (A): now also SW7.2; no longer SW7.1
- net at D62.2 (A): now also SW43.2; no longer SW43.1
- net at D100.2 (A): now also SW84.1; no longer SW84.2
- net at D107.2 (A): now also SW91.1; no longer SW91.2
- net at LED24.A: now also R63.1; no longer R63.2
- net at LED25.A: now also R64.1; no longer R64.2
- net at LED26.A: now also R65.1; no longer R65.2
- net at LED27.A: now also R66.1; no longer R66.2
- net at LED28.A: now also R67.1; no longer R67.2
- net at LED29.A: now also R68.1; no longer R68.2
- net at LED30.A: now also R69.1; no longer R69.2
- net at LED31.A: now also R70.1; no longer R70.2
- net at LED32.A: now also R71.1; no longer R71.2
- net at LED33.A: now also R72.1; no longer R72.2
- net at LED34.A: now also R73.1; no longer R73.2
- net at LED35.A: now also R74.1; no longer R74.2
- net at R80.1: now also Q3.3 (D)
- net at Q1.1 (G): now also R41.2
- net Col16 renamed C15
- net Col17 renamed C16
- net Col18 renamed C17
- net Col19 renamed C18
- removed net Col2: SW101.1, SW111.2, SW22.1, SW3.1, SW43.2, SW63.1, SW84.1
- removed net Col6: SW102.1, SW113.2, SW26.1, SW47.1, SW67.1, SW7.2, SW88.1
- removed net Col9: SW10.1, SW29.1, SW50.1, SW70.1, SW91.1
- net E-PB0: no longer names the net of U3.26 (PB0/TIM3_CH3)
- net E-PB10: no longer names the net of U3.29 (PB10/TIM2_CH3/SPI2_SCK/I2C2_SCL/I2S2_CK)
- net E-PC4: no longer names the net of U3.24 (PC4)
- net E-PC5: no longer names the net of U3.25 (PC5)
- net R6: no longer names the net of U3.10 (PC2/SPI2_MISO)
- new net: LED1.K, R59.1
- new net: LED2.K, R60.1
- new net: LED3.K, R61.1
- new net: LED43.K, R102.1
- new net: Q2.3 (D), R40.1, R41.1
- new net: Q2.1 (G), R42.2, R43.2
- new net: Q3.1 (G), R100.2, R83.2
Other:
- moved on the sheet: LED1, LED2, LED20, LED21, LED3, LED43, R102, R59, R60, R61, R80, SW43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

Commit message: Routing
Parts:
- added C14: 100n, Capacitor_SMD:C_0402_1005Metric, symbol Device:C_Small
- added Q1, Q2, Q3: 2N7002, Package_TO_SOT_SMD:SOT-23, symbol Transistor_FET:2N7002
- added R19, R21, R23: 100, Resistor_SMD:R_0402_1005Metric, symbol Device:R_Small
- added R20, R22, R24: 10k, Resistor_SMD:R_0402_1005Metric, symbol Device:R_Small
- added U4: AT24C256C-SSHL-T, acheron_Components:SOIC-8, symbol Memory_EEPROM:24LC256
- renumbered C14 to C15, C15 to C16, C16 to C17, C17 to C18, C18 to C19, C19 to C20, C20 to C21, C21 to C22, C22 to C23, C23 to C24, C24 to C25, C25 to C26, C26 to C27, C27 to C28, C28 to C29, C29 to C30, C30 to C31, C31 to C32, C32 to C33, C33 to C34, C34 to C35, C35 to C36, C36 to C37, C37 to C38, C38 to C39, Q1 to Q4, Q2 to Q5, Q3 to Q6, R94 to R100, R95 to R101, R96 to R102, R97 to R103, R98 to R104, R99 to R105, R100 to R106, R101 to R107, R102 to R108, R103 to R109, R104 to R110, R105 to R111, R106 to R112, R107 to R113, R108 to R114, R109 to R115, R110 to R116, R111 to R117, R112 to R118, R113 to R119, R114 to R120, R115 to R121, R116 to R122, R117 to R123, R118 to R124, R119 to R125, R120 to R126, R121 to R127, R122 to R128, R123 to R129, R124 to R130, R125 to R131, R126 to R132, R127 to R133, R128 to R134, R129 to R135, R130 to R136, R131 to R137, R132 to R138, R133 to R139, R134 to R140, R135 to R141, R136 to R142, R137 to R143, R138 to R144, R139 to R145, R140 to R146, R141 to R147, R142 to R148, R143 to R149, R144 to R150, R145 to R151, R146 to R152, R147 to R153, R148 to R154, R149 to R155, R150 to R156, R151 to R157, R19 to R25, R20 to R26, R21 to R27, R22 to R28, R23 to R29, R24 to R30, R25 to R31, R26 to R32, R27 to R33, R28 to R34, R29 to R35, R30 to R36, R31 to R37, R32 to R38, R33 to R39, R34 to R40, R35 to R41, R36 to R42, R37 to R43, R38 to R44, R39 to R45, R40 to R46, R41 to R47, R42 to R48, R43 to R49, R44 to R50, R45 to R51, R46 to R52, R47 to R53, R48 to R54, R49 to R55, R50 to R56, R51 to R57, R52 to R58, R53 to R59, R54 to R60, R55 to R61, R56 to R62, R57 to R63, R58 to R64, R59 to R65, R60 to R66, R61 to R67, R62 to R68, R63 to R69, R64 to R70, R65 to R71, R66 to R72, R67 to R73, R68 to R74, R69 to R75, R70 to R76, R71 to R77, R72 to R78, R73 to R79, R74 to R80, R75 to R81, R76 to R82, R77 to R83, R78 to R84, R79 to R85, R80 to R86, R81 to R87, R82 to R88, R83 to R89, R84 to R90, R85 to R91, R86 to R92, R87 to R93, R88 to R94, R89 to R95, R90 to R96, R91 to R97, R92 to R98, R93 to R99, U4 to U5, U5 to U6
Connections:
- net 3V3: now also C14.2, U4.8 (VCC)
- net C0: now also U3.20 (PA4/USART2_CK); no longer U3.21 (PA5/TIM2_CH1/SPI1_SCK)
- net C1: now also U3.17 (PA3/TIM2_CH4/USART2_RX); no longer U3.20 (PA4/USART2_CK)
- net C10: now also SW93.2, U3.61 (I2C1_SCL/TIM4_CH3/TIM10_CH1/PB8); no longer SW93.1
- net C11: now also U3.57 (SPI1_MOSI/SPI3_MOSI/TIM3_CH2/PB5)
- net C12: now also SW105.2, U3.50 (JTDI/TIM2_CH1/PA14); no longer SW105.1
- net C13: now also U3.10 (PC2/SPI2_MISO)
- net C14: now also U3.9 (PC1)
- net C15: now also U3.8 (PC0)
- net C2: now also U3.16 (PA2/TIM2_CH3/USART2_TX); no longer U3.17 (PA3/TIM2_CH4/USART2_RX)
- net C3: now also U3.15 (PA1/TIM2_CH2/USART2_RTS); no longer U3.16 (PA2/TIM2_CH3/USART2_TX)
- net C4: now also U3.14 (PA0/TIM2_CH1/USART2_CTS); no longer U3.15 (PA1/TIM2_CH2/USART2_RTS)
- net C5: no longer U3.14 (PA0/TIM2_CH1/USART2_CTS)
- net C6: now also SW89.2, U3.38 (USART6_RX/TIM3_CH2/PC7); no longer SW89.1, U3.37 (I2S2_MCK/TIM3_CH1/USART6_TX/PC6)
- net C7: now also U3.37 (I2S2_MCK/TIM3_CH1/USART6_TX/PC6); no longer U3.33 (PB12)
- net C8: now also U3.43 (USART1_RX/TIM1_CH3/PA10); no longer U3.41 (USART1_CK/TIM1_CH1/PA8)
- net CAPS_INDICATOR: now also R89.1, U3.39 (USART6_CK/TIM3_CH3/PC8); no longer U3.43 (USART1_RX/TIM1_CH3/PA10)
- net GND: now also R119.2, R135.2, R136.2, C14.1, Q1.2 (S), Q2.2 (S), Q3.2 (S), R20.1, R22.1, R24.1, U4.1 (A0), U4.2 (A1), U4.3 (A2), U4.4 (GND), U4.7 (WP); no longer LED72.K, LED93.K, LED94.K
- net INDICATOR1: now also U3.54 (PD2), R19.1; no longer R16.2
- net INDICATOR2: now also U3.55 (JTDO-SWO/SPI1_SCK/SPI3_SCK/I2C2_SDA/TIM2_CH2/PB3), R21.1; no longer R17.1
- net INDICATOR3: now also U3.56 (NJTRST/SPI1_MISO/SPI3_MISO/I2C3_SDA/TIM3_CH1/PB4), R23.1; no longer R18.1, R89.1, U3.38 (USART6_RX/TIM3_CH2/PC7)
- net LED_PWM: now also U3.26 (PB0/TIM3_CH3); no longer U3.27 (PB1/TIM3_CH4)
- net LED_SIGNAL: now also LED72.A, LED93.A, LED94.A; no longer R119.1, R135.1, R136.1
- net R0: now also U3.23 (PA7/SPI1_MOSI/TIM3_CH2)
- net R1: now also U3.24 (PC4)
- net R2: now also U3.25 (PC5)
- net R3: now also U3.27 (PB1/TIM3_CH4)
- net R4: now also U3.21 (PA5/TIM2_CH1/SPI1_SCK), U3.33 (PB12), U3.41 (USART1_CK/TIM1_CH1/PA8), U3.62 (I2C1_SDA/TIM4_CH4/TIM11_CH1/PB9)
- net R5: now also U3.11 (PC3/SPI2_MOSI), U3.22 (PA6/TIM3_CH1/SPI1_MISO)
- net SCL: now also U4.6 (SCL)
- net SDA: now also U4.5 (SDA)
- net at R16.1: now also LEDNUM1.K; no longer LEDSCR1.K
- net at R17.2: now also LEDCAPS1.K; no longer LEDNUM1.K
- net at R18.2: now also LEDSCR1.K; no longer LEDCAPS1.K
- net at D105.2 (A): now also SW89.1; no longer SW89.2
- net at D109.2 (A): now also SW93.1; no longer SW93.2
- net at D122.2 (A): now also SW105.1; no longer SW105.2
- new net: Q1.3 (D), R16.2
- new net: Q2.3 (D), R17.1
- new net: Q3.3 (D), R18.1
- new net: LED72.K, R119.1
- new net: LED93.K, R135.1
- new net: LED94.K, R136.1
- new net: Q2.1 (G), R21.2, R22.2
- new net: Q3.1 (G), R23.2, R24.2
- new net: Q1.1 (G), R19.2, R20.2
Other:
- note added: "EEPROM"
- note removed: ".>"
- note removed: "<,"
- note removed: "Shift"
- note removed: "Up"
- moved on the sheet: LED72, LED93, LED94, LEDCAPS1, LEDNUM1, LEDSCR1, R119, R135, R136, R16, R17, R18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

Commit message: Routing
Parts:
- removed X1: ARM JTAG, acheron_Connectors:PinHeader_2x5_P2.54mm_Vertical_Staggered, symbol Connector_Generic:Conn_02x05_Odd_Even
Connections:
- net 3V3: now also R11.1, R12.1; no longer R11.2, R12.2
- net C15: now also U3.53 (SPI3_MOSI/PC12)
- net C16: now also U3.52 (SPI3_MISO/PC11)
- net C17: now also U3.51 (SPI3_SCK/I2S3_CK/PC10)
- net GND: now also R145.2, R146.2; no longer LED101.K, LED102.K, LED103.K
- net LED_SIGNAL: now also LED101.A, LED102.A, LED103.A; no longer R145.1, R146.1
- net SCL: now also R12.2; no longer R12.1
- net SDA: now also R11.2; no longer R11.1
- new net: LED101.K, LED102.K, R145.1
- new net: LED103.K, R146.1
Other:
- moved on the sheet: LED101, LED102, LED103, R11, R145, R146

Commit message: Most routing, run some DRC, label missing
Parts:
- added X?: Conn_01x09, acheron_Connectors:PinHeader_1x10_P2.54mm_Vertical, symbol Connector_Generic:Conn_01x10
- renumbered D110 to D100, D111 to D101, D112 to D102, D113 to D103, D114 to D104, D115 to D105, D120 to D106, D121 to D107, D122 to D108, D123 to D109, D124 to D110, D125 to D111, D126 to D112, D127 to D113, D107 to D114, D108 to D115, D99 to D116, D100 to D117, D101 to D118, D102 to D119, D103 to D120, D104 to D121, D105 to D122, D106 to D123, D116 to D124, D117 to D125, D118 to D126, D119 to D127, D109 to D99, J1 to J2, LED101 to LED100, LED102 to LED101, LED103 to LED102, LED104 to LED103, LED105 to LED104, LED106 to LED105, LED107 to LED106, LED100 to LED107, LED68 to LED62, LED69 to LED63, LED71 to LED64, LED72 to LED65, LED62 to LED66, LED63 to LED67, LED64 to LED68, LED65 to LED69, LED66 to LED70, LED67 to LED71, LED70 to LED72, LED89 to LED81, LED90 to LED82, LED92 to LED83, LED93 to LED84, LED94 to LED85, LED81 to LED86, LED82 to LED87, LED83 to LED88, LED84 to LED89, LED85 to LED90, LED86 to LED91, LED87 to LED92, LED88 to LED93, LED91 to LED94, R117 to R115, R120 to R116, R121 to R117, R122 to R118, R123 to R119, R124 to R120, R125 to R121, R115 to R122, R116 to R123, R118 to R124, R119 to R125, R133 to R131, R137 to R132, R138 to R133, R139 to R134, R140 to R135, R131 to R136, R132 to R137, R134 to R138, R135 to R139, R136 to R140, R150 to R145, R151 to R146, R152 to R147, R153 to R148, R154 to R149, R155 to R150, R156 to R151, R145 to R152, R146 to R153, R147 to R154, R148 to R155, R149 to R156, SW81 to SW100, SW83 to SW101, SW84 to SW102, SW85 to SW103, SW86 to SW104, SW87 to SW105, SW88 to SW106, SW89 to SW107, SW90 to SW108, SW100 to SW109, SW101 to SW110, SW102 to SW111, SW110 to SW112, SW111 to SW113, SW112 to SW114, SW113 to SW115, SW82 to SW81, SW93 to SW82, SW94 to SW83, SW95 to SW84, SW96 to SW85, SW97 to SW86, SW98 to SW87, SW99 to SW88, SW103 to SW89, SW104 to SW90, SW105 to SW91, SW106 to SW92, SW107 to SW93, SW108 to SW94, SW109 to SW95, SW114 to SW96, SW115 to SW97, SW91 to SW98, SW92 to SW99, X2 to X1
Connections:
- net 3V3: now also X?.1 (Pin_1)
- net 5V: now also X?.8 (Pin_8)
- net C7: now also U3.33 (PB12); no longer U3.37 (I2S2_MCK/TIM3_CH1/USART6_TX/PC6)
- net E-PA9: now also X?.4 (Pin_4)
- net E-PB13: now also X?.3 (Pin_3)
- net E-PB14: now also X?.2 (Pin_2)
- net E-PC13: now also X?.5 (Pin_5)
- net E-PC14: now also X?.6 (Pin_6)
- net E-PC15: now also X?.7 (Pin_7)
- net GND: now also R122.2, R123.2, R124.2, R136.1, R137.2, R138.2, R154.2, R155.2, R156.2, X?.10 (Pin_10); no longer LED103.K, LED104.K, LED105.K, LED106.K, LED62.K, LED63.K, LED64.K, LED81.K, LED82.K, LED83.K
- net LED_SIGNAL: now also LED103.A, LED104.A, LED105.A, LED106.A, LED62.A, LED63.A, LED64.A, LED81.A, LED82.A, LED83.A; no longer R122.1, R123.1, R124.1, R136.1, R137.1, R138.1, R154.1, R155.1, R156.1
- net R4: no longer D114.1 (K), D115.1 (K), D116.1 (K), D117.1 (K), D118.1 (K), D119.1 (K), D120.1 (K), D121.1 (K), D122.1 (K), D123.1 (K), U3.21 (PA5/TIM2_CH1/SPI1_SCK), U3.33 (PB12), U3.41 (USART1_CK/TIM1_CH1/PA8)
- net R5: no longer D124.1 (K), D125.1 (K), D126.1 (K), D127.1 (K), U3.22 (PA6/TIM3_CH1/SPI1_MISO)
- net at R136.2: now also LED81.K; no longer LED81.A
- net R8: now reaches U3.29 (PB10/TIM2_CH3/SPI2_SCK/I2C2_SCL/I2S2_CK)
- net R8: now also D122.1 (K), D123.1 (K)
- new net: LED103.K, LED104.K, R154.1
- new net: LED62.K, R122.1
- new net: LED63.K, R123.1
- new net: LED64.K, R124.1
- new net: LED82.K, R137.1
- new net: LED83.K, R138.1
- new net: LED105.K, R155.1
- new net: LED106.K, R156.1
- new net E-PC6: U3.37 (I2S2_MCK/TIM3_CH1/USART6_TX/PC6), X?.9 (Pin_9)
- new net R6: D114.1 (K), D115.1 (K), U3.41 (USART1_CK/TIM1_CH1/PA8)
- new net R7: D116.1 (K), D117.1 (K), D118.1 (K), D119.1 (K), D120.1 (K), D121.1 (K), U3.21 (PA5/TIM2_CH1/SPI1_SCK)
- new net R9: D124.1 (K), D125.1 (K), D126.1 (K), D127.1 (K), U3.22 (PA6/TIM3_CH1/SPI1_MISO)
Other:
- note removed: "Switch matrix"
- moved on the sheet: D114, D115, D116, D117, D118, D119, D120, D121, D122, D123, D124, D125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

Commit message: New label, remove Acheron logo, add gondo logo
Parts:
- removed L3: OSHLogo, acheron_Graphics:osh-logo, symbol Mechanical:MountingHole
- added GR6: Warning sign, acheron_Graphics:Warning_Sign_3.6x3.2mm, symbol Mechanical:MountingHole
- L2: value LogoBack -> Gondolindrim Logo; footprint acheron_Logos:acheronLong -> gondolindrim_kicad_logos:gondolindrim_circuit-tree_50x15mm
- gave numbers to parts that had none: 1
- renumbered J2 to J1, L4 to L3, L5 to L4, X1 to X2
Connections:
- net C14: now also SW76.2; no longer SW76.1
- net at D94.2 (A): now also SW76.1; no longer SW76.2
Other:
- moved on the sheet: SW76

Commit message: Organize schematic
Parts:
- C18, C19, C20, C21, C22, C23, C24, C25, C26, C27, C28, C29, C30, C31, C32, C33, C34, C35, C36, C37, C38, C39: Manufacturer (none) -> Samsung; Manufacturer Part Number (none) -> CL05B104KB54PNC; Specification (none) -> 50V 100nF X7R ±10% 0402 MLCC; Vendor Part Number (none) -> LCSC C307331
- C9: Specification 16V 10uF Tantallum -> 16V 10uF CASEA Tantallum
- D10, D11, D12, D13, D14, D15, D16, D17, D18, D19, D20, D21, D22, D3, D4, D5, D6, D7, D8, D9: value WS2812C -> WS2812B-V5/W; LCSC Part Number C114587 -> (none); Vendor Part Number (none) -> LCSC C2874885
- D100, D101, D102, D103, D104, D105, D106, D107, D108, D109, D110, D111, D112, D113, D114, D115, D116, D117, D118, D119, D120, D121, D122, D123, D124, D125, D126, D127, D23, D24, D25, D26, D27, D28, D29, D30, D31, D32, D33, D34, D35, D36, D37, D38, D39, D40, D41, D42, D43, D44, D45, D46, D47, D48, D49, D50, D51, D52, D53, D54, D55, D56, D57, D58, D59, D60, D61, D62, D63, D64, D65, D66, D67, D68, D69, D70, D71, D72, D73, D74, D75, D76, D77, D78, D79, D80, D81, D82, D83, D84, D85, D86, D87, D88, D89, D90, D91, D92, D93, D94, D95, D96, D97, D98, D99: Manufacturer (none) -> Semtech; Specification (none) -> SOD-123 small signal switching diode; Vendor Part Number (none) -> LCSC C81598
- FB1: LCSC Part Number C139197 -> (none); Vendor Part Number (none) -> LCSC C139197
- J1: LCSC Part Number C2760486 -> (none); Vendor Part Number (none) -> LCSC C2760486
- R100, R101, R102, R103, R104, R105, R107, R108, R109, R110, R111, R112, R113, R114, R115, R116, R117, R118, R119, R120, R121, R122, R123, R124, R125, R126, R127, R128, R129, R130, R131, R132, R133, R134, R135, R136, R137, R138, R139, R140, R141, R142, R143, R144, R145, R146, R147, R148, R149, R150, R151, R152, R153, R154, R155, R156, R157, R16, R17, R18, R50, R51, R52, R53, R54, R55, R56, R57, R58, R59, R60, R61, R62, R63, R64, R65, R66, R67, R68, R69, R70, R71, R72, R73, R74, R75, R76, R77, R78, R79, R80, R81, R82, R83, R84, R85, R86, R87, R88, R90, R91, R92, R93, R94, R95, R96, R97, R98, R99: Manufacturer (none) -> Uniroyal; Manufacturer Part Number (none) -> 0402WGF1001TCE; Specification (none) -> ±1% 1/16W Thick Film Resistors 50V 0402; Vendor Part Number (none) -> LCSC C11702
- R14, R15: Manufacturer (none) -> Uniroyal; Manufacturer Part Number (none) -> 0402WGF5101TCE; Specification (none) -> ±1% 1/16W Thick Film Resistors 50V 0402; Vendor Part Number (none) -> LCSC C25905
- R25, R26, R27, R28, R29, R30, R31, R32, R33, R34, R35, R36, R37, R38, R39, R40, R41, R42, R43, R44: Manufacturer (none) -> Uniroyal; Manufacturer Part Number (none) -> 0402WGF510KTCE; Specification (none) -> ±1% 1/16W Thick Film Resistors 50V 0402; Vendor Part Number (none) -> LCSC C25128
- R45: Manufacturer (none) -> Uniroyal; Manufacturer Part Number (none) -> 0402WGF1002TCE; Specification (none) -> ±1% 1/16W Thick Film Resistors 50V 0402; Vendor Part Number (none) -> LCSC C25744
- U5: LCSC Part Number C138714 -> (none); Vendor Part Number (none) -> LCSC C138714
- U6: LCSC Part Number C132604 -> (none); Vendor Part Number (none) -> LCSC C132604
- renumbered L3 to GR?, L1 to GR?, L2 to GR?, L4 to GR?
Other:
- note added: "GRAPHICS"
- note removed: "Indicator lights"
- note removed: "Logos and flags"
- moved on the sheet: GR1, GR2, GR3, GR4, GR5, GR6, LED1, LED10, LED100, LED101, LED102, LED103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
