File: kicad_files/austin.kicad_sch (KiCad schematic)
At the start: 582 parts, among them J1 TYPE-C-31-M-12, Q1 2N7002, Q2 2N7002, Q3 2N7002, Q4 AO3401A, Q5 2N7002, Q6 2N7002, SW1 K2-1187SQ-A4SW-06, SW10 Mechanical_Switch, SW100 Mechanical_Switch, SW101 Mechanical_Switch, SW102 Mechanical_Switch, SW103 Mechanical_Switch, SW104 Mechanical_Switch, SW105 Mechanical_Switch, SW106 Mechanical_Switch, SW107 Mechanical_Switch, SW108 Mechanical_Switch, SW109 Mechanical_Switch, SW11 Mechanical_Switch, SW110 Mechanical_Switch, SW111 Mechanical_Switch, SW112 Mechanical_Switch, SW113 Mechanical_Switch, SW114 Mechanical_Switch, SW115 Mechanical_Switch, SW12 Mechanical_Switch, SW13 Mechanical_Switch, SW14 Mechanical_Switch, SW15 Mechanical_Switch, SW16 Mechanical_Switch, SW17 Mechanical_Switch, SW18 Mechanical_Switch, SW19 Mechanical_Switch, SW2 Mechanical_Switch, SW20 Mechanical_Switch, SW21 Mechanical_Switch, SW22 Mechanical_Switch, SW23 Mechanical_Switch, SW24 Mechanical_Switch, SW25 Mechanical_Switch, SW26 Mechanical_Switch, SW27 Mechanical_Switch, SW28 Mechanical_Switch, SW29 Mechanical_Switch, SW3 Mechanical_Switch, SW30 Mechanical_Switch, SW31 Mechanical_Switch, SW32 Mechanical_Switch, SW33 Mechanical_Switch, SW34 Mechanical_Switch, SW35 Mechanical_Switch, SW36 Mechanical_Switch, SW37 Mechanical_Switch, SW38 Mechanical_Switch, SW39 Mechanical_Switch, SW4 Mechanical_Switch, SW40 Mechanical_Switch, SW41 Mechanical_Switch, SW42 Mechanical_Switch, SW43 Mechanical_Switch, SW44 Mechanical_Switch, SW45 Mechanical_Switch, SW46 Mechanical_Switch, SW47 Mechanical_Switch, SW48 Mechanical_Switch, SW49 Mechanical_Switch, SW5 Mechanical_Switch, SW50 Mechanical_Switch, SW51 Mechanical_Switch, SW52 Mechanical_Switch, SW53 Mechanical_Switch, SW54 Mechanical_Switch, SW55 Mechanical_Switch, SW56 Mechanical_Switch, SW57 Mechanical_Switch, SW58 Mechanical_Switch, SW59 Mechanical_Switch, SW6 Mechanical_Switch, SW60 Mechanical_Switch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

Commit message: Fix column pin assortment, review USB routing
Parts:
- added F1: nSMD100-16V, Fuse:Fuse_1206_3216Metric, symbol Device:Fuse
- X1: value Conn_01x09 -> EXTRA_PINS; now in the parts list
- gave numbers to parts that had none: 4
- renumbered C6 to C1, C12 to C10, C13 to C11, C14 to C12, C15 to C13, C16 to C14, C17 to C15, C4 to C16, C5 to C17, C7 to C2, C8 to C3, C9 to C4, C1 to C5, C2 to C6, C3 to C7, C10 to C8, C11 to C9, GR6 to GR10, GR2 to GR3, GR3 to GR5, GR4 to GR7, GR5 to GR9, LED20 to LED1, LED8 to LED10, LED9 to LED11, LED10 to LED12, LED11 to LED13, LED12 to LED14, LED13 to LED15, LED14 to LED16, LED15 to LED17, LED16 to LED18, LED17 to LED19, LED21 to LED2, LED18 to LED20, LED19 to LED21, LED1 to LED3, LED2 to LED4, LED3 to LED5, LED4 to LED6, LED5 to LED7, LED6 to LED8, LED7 to LED9, Q6 to Q4, Q4 to Q5, Q5 to Q6, R11 to R1, R14 to R10, R99 to R100, R100 to R101, R101 to R102, R102 to R103, R103 to R104, R104 to R105, R105 to R106, R7 to R11, R15 to R12, R8 to R13, R9 to R14, R10 to R15, R86 to R19, R12 to R2, R19 to R20, R20 to R21, R21 to R22, R22 to R23, R89 to R24, R23 to R25, R24 to R26, R106 to R27, R25 to R28, R26 to R29, R13 to R3, R27 to R30, R28 to R31, R29 to R32, R30 to R33, R31 to R34, R32 to R35, R33 to R36, R34 to R37, R35 to R38, R36 to R39, R1 to R4, R37 to R40, R38 to R41, R39 to R42, R40 to R43, R41 to R44, R42 to R45, R43 to R46, R44 to R47, R45 to R48, R46 to R49, R2 to R5, R47 to R50, R48 to R51, R49 to R52, R50 to R53, R51 to R54, R52 to R55, R53 to R56, R54 to R57, R55 to R58, R56 to R59, R3 to R6, R57 to R60, R58 to R61, R59 to R62, R60 to R63, R61 to R64, R62 to R65, R63 to R66, R64 to R67, R65 to R68, R66 to R69, R4 to R7, R67 to R70, R68 to R71, R69 to R72, R70 to R73, R71 to R74, R72 to R75, R73 to R76, R74 to R77, R75 to R78, R76 to R79, R5 to R8, R77 to R80, R78 to R81, R79 to R82, R80 to R83, R81 to R84, R82 to R85, R83 to R86, R84 to R87, R85 to R88, R87 to R89, R6 to R9, R88 to R90, R90 to R91, R91 to R92, R92 to R93, R93 to R94, R94 to R95, R95 to R96, R96 to R97, R97 to R98, R98 to R99, U3 to U1, U1 to U2, U4 to U3, U2 to U4
Connections:
- net 5V: now also C5.2, R4.2, F1.1; no longer C5.1, R4.1
- net C0: now also U1.21 (PA5/TIM2_CH1/SPI1_SCK); no longer U1.20 (PA4/USART2_CK)
- net C1: now also U1.20 (PA4/USART2_CK); no longer U1.17 (PA3/TIM2_CH4/USART2_RX)
- net C13: now also U1.9 (PC1); no longer U1.10 (PC2/SPI2_MISO)
- net C14: now also U1.8 (PC0); no longer U1.9 (PC1)
- net C15: no longer U1.8 (PC0)
- net C18: now also U1.11 (PC3/SPI2_MOSI)
- net C2: now also U1.17 (PA3/TIM2_CH4/USART2_RX); no longer U1.16 (PA2/TIM2_CH3/USART2_TX)
- net C3: now also U1.16 (PA2/TIM2_CH3/USART2_TX); no longer U1.15 (PA1/TIM2_CH2/USART2_RTS)
- net C4: now also U1.15 (PA1/TIM2_CH2/USART2_RTS); no longer U1.14 (PA0/TIM2_CH1/USART2_CTS)
- net C5: now also U1.14 (PA0/TIM2_CH1/USART2_CTS)
- net C6: now also U1.37 (I2S2_MCK/TIM3_CH1/USART6_TX/PC6); no longer U1.38 (USART6_RX/TIM3_CH2/PC7)
- net E-PC6: no longer U1.37 (I2S2_MCK/TIM3_CH1/USART6_TX/PC6)
- net GND: now also C5.1, R4.1; no longer C5.2, R4.2
- net LED_PWM: now also U1.27 (PB1/TIM3_CH4); no longer U1.26 (PB0/TIM3_CH3)
- net R0: now also U1.24 (PC4); no longer U1.23 (PA7/SPI1_MOSI/TIM3_CH2)
- net R1: now also U1.25 (PC5); no longer U1.24 (PC4)
- net R2: now also U1.26 (PB0/TIM3_CH3); no longer U1.25 (PC5)
- net R3: now also U1.38 (USART6_RX/TIM3_CH2/PC7); no longer U1.27 (PB1/TIM3_CH4)
- net R5: now also U1.10 (PC2/SPI2_MISO); no longer U1.11 (PC3/SPI2_MOSI)
- net R7: now also U1.22 (PA6/TIM3_CH1/SPI1_MISO); no longer U1.21 (PA5/TIM2_CH1/SPI1_SCK)
- net R9: now also U1.23 (PA7/SPI1_MOSI/TIM3_CH2); no longer U1.22 (PA6/TIM3_CH1/SPI1_MISO)
- net VBUS: now also F1.2
Other:
- moved on the sheet: C1, C10, C11, C13, C14, C15, C16, C17, C2, C3, C4, C5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
