File: kicad_files/austin.kicad_sch (KiCad schematic)
At the start: 583 parts, among them J1 TYPE-C-31-M-12, Q1 2N7002, Q2 2N7002, Q3 2N7002, Q4 2N7002, Q5 AO3401A, Q6 2N7002, SW1 K2-1187SQ-A4SW-06, SW10 Mechanical_Switch, SW100 Mechanical_Switch, SW101 Mechanical_Switch, SW102 Mechanical_Switch, SW103 Mechanical_Switch, SW104 Mechanical_Switch, SW105 Mechanical_Switch, SW106 Mechanical_Switch, SW107 Mechanical_Switch, SW108 Mechanical_Switch, SW109 Mechanical_Switch, SW11 Mechanical_Switch, SW110 Mechanical_Switch, SW111 Mechanical_Switch, SW112 Mechanical_Switch, SW113 Mechanical_Switch, SW114 Mechanical_Switch, SW115 Mechanical_Switch, SW12 Mechanical_Switch, SW13 Mechanical_Switch, SW14 Mechanical_Switch, SW15 Mechanical_Switch, SW16 Mechanical_Switch, SW17 Mechanical_Switch, SW18 Mechanical_Switch, SW19 Mechanical_Switch, SW2 Mechanical_Switch, SW20 Mechanical_Switch, SW21 Mechanical_Switch, SW22 Mechanical_Switch, SW23 Mechanical_Switch, SW24 Mechanical_Switch, SW25 Mechanical_Switch, SW26 Mechanical_Switch, SW27 Mechanical_Switch, SW28 Mechanical_Switch, SW29 Mechanical_Switch, SW3 Mechanical_Switch, SW30 Mechanical_Switch, SW31 Mechanical_Switch, SW32 Mechanical_Switch, SW33 Mechanical_Switch, SW34 Mechanical_Switch, SW35 Mechanical_Switch, SW36 Mechanical_Switch, SW37 Mechanical_Switch, SW38 Mechanical_Switch, SW39 Mechanical_Switch, SW4 Mechanical_Switch, SW40 Mechanical_Switch, SW41 Mechanical_Switch, SW42 Mechanical_Switch, SW43 Mechanical_Switch, SW44 Mechanical_Switch, SW45 Mechanical_Switch, SW46 Mechanical_Switch, SW47 Mechanical_Switch, SW48 Mechanical_Switch, SW49 Mechanical_Switch, SW5 Mechanical_Switch, SW50 Mechanical_Switch, SW51 Mechanical_Switch, SW52 Mechanical_Switch, SW53 Mechanical_Switch, SW54 Mechanical_Switch, SW55 Mechanical_Switch, SW56 Mechanical_Switch, SW57 Mechanical_Switch, SW58 Mechanical_Switch, SW59 Mechanical_Switch, SW6 Mechanical_Switch, SW60 Mechanical_Switch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

Commit message: Switch matrix rework, organize schematic
- The switch matrix was reorganized so the ISO keys and ANSI keys are separated; this should give ISO users a friendlier usage as they will not need to reconfigure keys once they use the keyboard.
- Schematic was reorganized and designators reset. PCB was updated accordingly
Parts:
- removed GR9: Warning sign, acheron_Graphics:warning_sign_3.6x3.2mm, symbol Mechanical:MountingHole
- added D93, D99: 1N4148W, acheron_Components:D_SOD-123, symbol Device:D
- SW100: Keycode ANSISHIFT -> ANSI (225) SHIFT
- SW101: Keycode ISOSHIFT -> ISO (125) SHIFT
- SW54: renamed from SW41; Keycode ISOENTER -> ISO ENTER
- SW83: renamed from SW74; Keycode ANSIENTER -> ANSI ENTER
- SW93: Keycode LZERO -> L 1U ZERO
- SW94: Keycode RZERO -> R 1U ZERO
- X2: renamed from X1; now left out of the parts list
- renumbered C16 to C1, C21 to C10, C22 to C11, C23 to C12, C24 to C13, C25 to C14, C26 to C15, C27 to C16, C28 to C17, C29 to C18, C30 to C19, C17 to C2, C31 to C20, C32 to C21, C33 to C22, C34 to C23, C35 to C24, C36 to C25, C37 to C26, C38 to C27, C39 to C28, C1 to C29, C5 to C3, C2 to C30, C3 to C31, C4 to C32, C8 to C33, C9 to C34, C10 to C35, C11 to C36, C13 to C37, C14 to C38, C15 to C39, C6 to C4, C7 to C5, C12 to C6, C18 to C7, C19 to C8, C20 to C9, D2 to D1, D98 to D100, D99 to D101, D100 to D102, D101 to D103, D102 to D104, D103 to D105, D104 to D106, D105 to D107, D106 to D108, D107 to D109, D108 to D110, D109 to D111, D110 to D112, D111 to D113, D112 to D114, D113 to D115, D114 to D116, D115 to D117, D116 to D118, D117 to D119, D118 to D120, D119 to D121, D120 to D122, D121 to D123, D122 to D124, D123 to D125, D124 to D126, D125 to D127, D126 to D128, D127 to D129, D1 to D2, D93 to D94, D94 to D95, D95 to D96, D96 to D97, D97 to D98, GR10 to GR9, R6 to R1, R5 to R10, R103 to R100, R104 to R101, R105 to R102, R106 to R103, R107 to R104, R108 to R105, R109 to R106, R110 to R107, R111 to R108, R112 to R109, R10 to R11, R113 to R110, R114 to R111, R115 to R112, R116 to R113, R117 to R114, R118 to R115, R119 to R116, R120 to R117, R121 to R118, R122 to R119, R123 to R120, R124 to R121, R125 to R122, R126 to R123, R127 to R124, R128 to R125, R129 to R126, R130 to R127, R131 to R128, R132 to R129, R16 to R13, R133 to R130, R134 to R131, R135 to R132, R136 to R133, R137 to R134, R138 to R135, R139 to R136, R140 to R137, R141 to R138, R142 to R139, R17 to R14, R143 to R140, R144 to R141, R145 to R142, R146 to R143, R147 to R144, R148 to R145, R149 to R146, R150 to R147, R151 to R148, R152 to R149, R18 to R15, R153 to R150, R154 to R151, R155 to R152, R156 to R153, R157 to R154, R1 to R155, R2 to R156, R3 to R157, R19 to R16, R20 to R17, R21 to R18, R22 to R19, R7 to R2, R23 to R20, R24 to R21, R25 to R22, R26 to R23, R27 to R24, R28 to R25, R29 to R26, R30 to R27, R31 to R28, R32 to R29, R8 to R3, R33 to R30, R34 to R31, R35 to R32, R36 to R33, R37 to R34, R38 to R35, R39 to R36, R40 to R37, R41 to R38, R42 to R39, R9 to R4, R43 to R40, R44 to R41, R45 to R42, R46 to R43, R47 to R44, R48 to R45, R49 to R46, R50 to R47, R51 to R48, R52 to R49, R11 to R5, R53 to R50, R54 to R51, R55 to R52, R56 to R53, R57 to R54, R58 to R55, R59 to R56, R60 to R57, R61 to R58, R62 to R59, R13 to R6, R63 to R60, R64 to R61, R65 to R62, R66 to R63, R67 to R64, R68 to R65, R69 to R66, R70 to R67, R71 to R68, R72 to R69, R14 to R7, R73 to R70, R74 to R71, R75 to R72, R76 to R73, R77 to R74, R78 to R75, R79 to R76, R80 to R77, R81 to R78, R82 to R79, R15 to R8, R83 to R80, R84 to R81, R85 to R82, R86 to R83, R87 to R84, R88 to R85, R89 to R86, R90 to R87, R91 to R88, R92 to R89, R4 to R9, R93 to R90, R94 to R91, R95 to R92, R96 to R93, R97 to R94, R98 to R95, R99 to R96, R100 to R97, R101 to R98, R102 to R99, SW42 to SW41, SW43 to SW42, SW44 to SW43, SW45 to SW44, SW46 to SW45, SW47 to SW46, SW48 to SW47, SW49 to SW48, SW50 to SW49, SW51 to SW50, SW52 to SW51, SW53 to SW52, SW54 to SW53, SW56 to SW55, SW57 to SW56, SW58 to SW57, SW59 to SW58, SW60 to SW59, SW62 to SW60, SW63 to SW61, SW64 to SW62, SW65 to SW63, SW66 to SW64, SW67 to SW65, SW68 to SW66, SW69 to SW67, SW70 to SW68, SW71 to SW69, SW72 to SW70, SW73 to SW71, SW61 to SW72, SW75 to SW73, SW76 to SW74, SW77 to SW75, SW78 to SW76, SW79 to SW77, SW80 to SW78, SW55 to SW79, SW81 to SW80, SW82 to SW81, SW83 to SW82, U4 to U1, U5 to U4, U6 to U5, U1 to U6, X2 to X1
Connections:
- net C12: no longer SW80.1
- net C13: now also SW80.1; no longer SW73.1, SW84.1
- net C14: now also SW73.1, SW84.1; no longer SW74.2, SW85.1
- net C15: now also SW74.2, SW85.1; no longer SW75.1, SW86.1
- net C16: now also SW75.1, SW86.1; no longer SW76.1, SW87.1
- net C17: now also SW76.1, SW87.1; no longer SW77.1, SW88.1
- net C18: now also SW77.1, SW88.1
- net R3: now also D93.1 (K)
- net R4: now also D99.1 (K)
- net at D92.2 (A), SW72.2: no longer SW83.2
- net at D74.2 (A), SW54.2: no longer SW79.2
- new net: D99.2 (A), SW83.2
Other:
- note added: "INDICATORS"
- note added: "LED MATRIX"
- note added: "SWITCH MATRIX"
- note added: "USB"
- note removed: "(*) "Spooky pins": on STM32F4x1, pins A9 and B2 cannot be used for switch matrix: - A9 is meant to be used as a VBUS sensing. It has a undocumented internal pulldown resistor; - B2 is used as BOOT1 during bootup, so it needs an external pulldown for successful bootup"
- note removed: "(**) PA9 jumper: a solderable jumper used to tie PA9 to VBUS. It is disconnected by default, hence PA9 is left floating"
- note removed: "/?"
- note removed: "Note that the - key is next to *, but was placed here so that an extra column just for this switch would not be needed"
- note removed: "Switch LED matrix"
- note removed: "USB Connector"
- moved on the sheet: C1, C10, C11, C12, C13, C14, C15, C16, C17, C18, C19, C2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
